File: RJ45LVDS_SPI.sch (EAGLE design)
At the start: 44 parts, among them J1 RJHSE-3381, U1 SN65MLVD206, U2 SN65MLVD206, U3 SN65MLVD206, U4 SN65MLVD206, U5 SN74LVC1T45DBVR, U6 SN74LVC1T45DBVR, U7 SN74LVC1T45DBVR, U8 SN74LVC1T45DBVR, U9 MIC37100

Commit message: documentation update
Parts:
- removed C11: .1u, rcl-dhs:C-USC0603
- added R5: 100, rcl-dhs:R-US_R0603
- added SJ13: (no value), jumper:SJ
Connections:
- new net N$18: R5.2, SJ13.2
- new net N$19: J1.GRN+, R5.1
- net +3V3: now also SJ13.1
- net +5V: no longer C11.1
- net GND: no longer C11.2, J1.GRN+
Changed lines of the file:
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@@
 <part name="C3" library="rcl-dhs" deviceset="C-US" device="C0603" value=".1u"/>
 <part name="C4" library="rcl-dhs" deviceset="C-US" device="C0603" value=".1u"/>
-<part name="C11" library="rcl-dhs" deviceset="C-US" device="C0603" value=".1u"/>
 <part name="SUPPLY22" library="supply2" deviceset="GND" device=""/>
 <part name="+3V17" library="supply1" deviceset="+3V3" device=""/>
@@
 <part name="SUPPLY31" library="supply2" deviceset="GND" device=""/>
 <part name="SUPPLY34" library="supply2" deviceset="GND" device=""/>
-<part name="SUPPLY36" library="supply2" deviceset="GND" device=""/>
 <part name="C8" library="rcl-dhs" deviceset="C-US" device="C0603" value=".1u"/>
 <part name="SUPPLY28" library="supply2" deviceset="GND" device=""/>
@@
 <part name="SJ12" library="jumper" deviceset="SJ" device=""/>
 <part name="SUPPLY8" library="supply2" deviceset="GND" device=""/>
+<part name="SJ13" library="jumper" deviceset="SJ" device=""/>
+<part name="+3V5" library="supply1" deviceset="+3V3" device=""/>
+<part name="R5" library="rcl-dhs" deviceset="R-US_" device="R0603" value="100"/>
 </parts>
 <sheets>
@@
 <instance part="C3" gate="G$1" x="20.32" y="187.96"/>
 <instance part="C4" gate="G$1" x="27.94" y="187.96"/>
-<instance part="C11" gate="G$1" x="-33.02" y="144.78"/>
 <instance part="SUPPLY22" gate="GND" x="30.48" y="175.26"/>
 <instance part="+3V17" gate="G$1" x="-2.54" y="195.58" rot="R90"/>
@@
 <instance part="SUPPLY31" gate="GND" x="10.16" y="162.56" rot="R90"/>
 <instance part="SUPPLY34" gate="GND" x="180.34" y="50.8"/>
-<instance part="SUPPLY36" gate="GND" x="-33.02" y="137.16"/>
 <instance part="C8" gate="G$1" x="35.56" y="187.96"/>
 <instance part="SUPPLY28" gate="GND" x="-104.14" y="58.42"/>
@@
 <instance part="SJ12" gate="1" x="30.48" y="149.86"/>
 <instance part="SUPPLY8" gate="GND" x="162.56" y="78.74"/>
+<instance part="SJ13" gate="1" x="-139.7" y="68.58"/>
+<instance part="+3V5" gate="G$1" x="-152.4" y="81.28"/>
+<instance part="R5" gate="G$1" x="-127" y="68.58" rot="R180"/>
 </instances>
 <busses>
@@
 </segment>
 <segment>
-<pinref part="C11" gate="G$1" pin="2"/>
-<pinref part="SUPPLY36" gate="GND" pin="GND"/>
-</segment>
-<segment>
-<pinref part="J1" gate="G$1" pin="GRN+"/>
-<wire x1="-93.98" y1="73.66" x2="-104.14" y2="73.66" width="0.1524" layer="91"/>
-<wire x1="-104.14" y1="73.66" x2="-104.14" y2="71.12" width="0.1524" layer="91"/>
 <pinref part="J1" gate="G$1" pin="YEL-"/>
 <wire x1="-104.14" y1="71.12" x2="-104.14" y2="63.5" width="0.1524" layer="91"/>
@@
 <pinref part="J1" gate="G$1" pin="GRN-"/>
 <wire x1="-93.98" y1="71.12" x2="-104.14" y2="71.12" width="0.1524" layer="91"/>
-<junction x="-104.14" y="71.12"/>
 <pinref part="SUPPLY28" gate="GND" pin="GND"/>
 <junction x="-104.14" y="60.96"/>
@@
 <junction x="157.48" y="114.3"/>
 </segment>
+<segment>
+<pinref part="+3V5" gate="G$1" pin="+3V3"/>
+<wire x1="-152.4" y1="78.74" x2="-152.4" y2="68.58" width="0.1524" layer="91"/>
+<pinref part="SJ13" gate="1" pin="1"/>
+<wire x1="-152.4" y1="68.58" x2="-144.78" y2="68.58" width="0.1524" layer="91"/>
+</segment>
 </net>
 <net name="3_33" class="0">
@@
 <segment>
 <pinref part="C10" gate="G$1" pin="1"/>
-<wire x1="-33.02" y1="147.32" x2="-33.02" y2="152.4" width="0.1524" layer="91"/>
 <wire x1="-33.02" y1="152.4" x2="-30.48" y2="152.4" width="0.1524" layer="91"/>
 <label x="-25.4" y="154.94" size="1.778" layer="95"/>
@@
 <junction x="-30.48" y="152.4"/>
 <pinref part="P+1" gate="1" pin="+5V"/>
-<pinref part="C11" gate="G$1" pin="1"/>
 <wire x1="-20.32" y1="152.4" x2="-7.62" y2="152.4" width="0.1524" layer="91"/>
 <junction x="-20.32" y="152.4"/>
@@
 </segment>
 </net>
+<net name="N$18" class="0">
+<segment>
+<pinref part="SJ13" gate="1" pin="2"/>
+<pinref part="R5" gate="G$1" pin="2"/>
+<wire x1="-134.62" y1="68.58" x2="-132.08" y2="68.58" width="0.1524" layer="91"/>
+</segment>
+</net>
+<net name="N$19" class="0">
+<segment>
+<pinref part="J1" gate="G$1" pin="GRN+"/>
+<wire x1="-93.98" y1="73.66" x2="-116.84" y2="73.66" width="0.1524" layer="91"/>
+<wire x1="-116.84" y1="73.66" x2="-116.84" y2="68.58" width="0.1524" layer="91"/>
+<pinref part="R5" gate="G$1" pin="1"/>
+<wire x1="-116.84" y1="68.58" x2="-121.92" y2="68.58" width="0.1524" layer="91"/>
+</segment>
+</net>

Commit message: deleted backup files
Parts:
- R5: value 100 -> 750
- U9: value MIC37100 -> MIC39100-3.3WS
Changed lines of the file:
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@@
 <part name="R4" library="rcl-dhs" deviceset="R-US_" device="R0603" value="100"/>
 <part name="P+1" library="supply1" deviceset="+5V" device=""/>
-<part name="U9" library="dds-boards" deviceset="MIC37100" device=""/>
+<part name="U9" library="dds-boards" deviceset="MIC37100" device="" value="MIC39100-3.3WS"/>
 <part name="SUPPLY31" library="supply2" deviceset="GND" device=""/>
 <part name="SUPPLY34" library="supply2" deviceset="GND" device=""/>
@@
 <part name="SJ13" library="jumper" deviceset="SJ" device=""/>
 <part name="+3V5" library="supply1" deviceset="+3V3" device=""/>
-<part name="R5" library="rcl-dhs" deviceset="R-US_" device="R0603" value="100"/>
+<part name="R5" library="rcl-dhs" deviceset="R-US_" device="R0603" value="750"/>
 </parts>
 <sheets>

Commit message: tweaks
Parts:
- removed SJ13: (no value), jumper:SJ
Connections:
- removed net N$18: R5.2, SJ13.2
- net +3V3: now also R5.2; no longer SJ13.1
Changed lines of the file:
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@@
 <part name="SJ12" library="jumper" deviceset="SJ" device=""/>
 <part name="SUPPLY8" library="supply2" deviceset="GND" device=""/>
-<part name="SJ13" library="jumper" deviceset="SJ" device=""/>
 <part name="+3V5" library="supply1" deviceset="+3V3" device=""/>
 <part name="R5" library="rcl-dhs" deviceset="R-US_" device="R0603" value="750"/>
@@
 <instance part="SJ12" gate="1" x="30.48" y="149.86"/>
 <instance part="SUPPLY8" gate="GND" x="162.56" y="78.74"/>
-<instance part="SJ13" gate="1" x="-139.7" y="68.58"/>
 <instance part="+3V5" gate="G$1" x="-152.4" y="81.28"/>
 <instance part="R5" gate="G$1" x="-127" y="68.58" rot="R180"/>
@@
 <pinref part="+3V5" gate="G$1" pin="+3V3"/>
 <wire x1="-152.4" y1="78.74" x2="-152.4" y2="68.58" width="0.1524" layer="91"/>
-<pinref part="SJ13" gate="1" pin="1"/>
-<wire x1="-152.4" y1="68.58" x2="-144.78" y2="68.58" width="0.1524" layer="91"/>
+<pinref part="R5" gate="G$1" pin="2"/>
+<wire x1="-152.4" y1="68.58" x2="-132.08" y2="68.58" width="0.1524" layer="91"/>
 </segment>
 </net>
@@
 </segment>
 </net>
-<net name="N$18" class="0">
-<segment>
-<pinref part="SJ13" gate="1" pin="2"/>
-<pinref part="R5" gate="G$1" pin="2"/>
-<wire x1="-134.62" y1="68.58" x2="-132.08" y2="68.58" width="0.1524" layer="91"/>
-</segment>
-</net>

Commit message: Bom added
Parts:
- added C11: .1u, rcl-dhs:C-USC0603
- C10, C16, C9: device rcl-dhs:C-USC1206K -> rcl:CPOL-USSMCB
Connections:
- net +3V3: now also C9.+; no longer C9.1
- net +5V: now also C10.+, C11.1; no longer C10.1
- net GND: now also C10.-, C11.2, C16.-, C9.-; no longer C10.2, C16.2, C9.2
- net N$16: now also C16.+; no longer C16.1
Changed lines of the file:
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@@
 <part name="SUPPLY22" library="supply2" deviceset="GND" device=""/>
 <part name="+3V17" library="supply1" deviceset="+3V3" device=""/>
-<part name="C9" library="rcl-dhs" deviceset="C-US" device="C1206K" value="10u"/>
-<part name="C10" library="rcl-dhs" deviceset="C-US" device="C1206K" value="10u"/>
+<part name="C9" library="rcl" deviceset="CPOL-US" device="SMCB" value="10u"/>
+<part name="C10" library="rcl" deviceset="CPOL-US" device="SMCB" value="10u"/>
 <part name="SUPPLY23" library="supply2" deviceset="GND" device=""/>
 <part name="SUPPLY24" library="supply2" deviceset="GND" device=""/>
@@
 <part name="C15" library="rcl-dhs" deviceset="C-US" device="C0603" value=".1u"/>
 <part name="SUPPLY7" library="supply2" deviceset="GND" device=""/>
-<part name="C16" library="rcl-dhs" deviceset="C-US" device="C1206K" value="10u"/>
+<part name="C16" library="rcl" deviceset="CPOL-US" device="SMCB" value="10u"/>
 <part name="SJ12" library="jumper" deviceset="SJ" device=""/>
 <part name="SUPPLY8" library="supply2" deviceset="GND" device=""/>
 <part name="+3V5" library="supply1" deviceset="+3V3" device=""/>
 <part name="R5" library="rcl-dhs" deviceset="R-US_" device="R0603" value="750"/>
+<part name="C11" library="rcl-dhs" deviceset="C-US" device="C0603" value=".1u"/>
 </parts>
 <sheets>
@@
 <instance part="+3V5" gate="G$1" x="-152.4" y="81.28"/>
 <instance part="R5" gate="G$1" x="-127" y="68.58" rot="R180"/>
+<instance part="C11" gate="G$1" x="-33.02" y="149.86"/>
 </instances>
 <busses>
@@
 </segment>
 <segment>
-<pinref part="C9" gate="G$1" pin="2"/>
+<pinref part="C9" gate="G$1" pin="-"/>
 <pinref part="SUPPLY24" gate="GND" pin="GND"/>
 <wire x1="40.64" y1="137.16" x2="40.64" y2="139.7" width="0.1524" layer="91"/>
 </segment>
 <segment>
-<pinref part="C10" gate="G$1" pin="2"/>
+<pinref part="C10" gate="G$1" pin="-"/>
 <pinref part="SUPPLY25" gate="GND" pin="GND"/>
+<pinref part="C11" gate="G$1" pin="2"/>
+<wire x1="-33.02" y1="144.78" x2="-20.32" y2="144.78" width="0.1524" layer="91"/>
+<junction x="-20.32" y="144.78"/>
 </segment>
 <segment>
@@
 </segment>
 <segment>
-<pinref part="C16" gate="G$1" pin="2"/>
+<pinref part="C16" gate="G$1" pin="-"/>
 <pinref part="SUPPLY8" gate="GND" pin="GND"/>
 <wire x1="162.56" y1="83.82" x2="162.56" y2="81.28" width="0.1524" layer="91"/>
@@
 <pinref part="+3V17" gate="G$1" pin="+3V3"/>
 <junction x="0" y="195.58"/>
-<pinref part="C9" gate="G$1" pin="1"/>
+<pinref part="C9" gate="G$1" pin="+"/>
 <wire x1="40.64" y1="147.32" x2="40.64" y2="149.86" width="0.1524" layer="91"/>
 <wire x1="40.64" y1="149.86" x2="40.64" y2="165.1" width="0.1524" layer="91"/>
@@
 <net name="+5V" class="0">
 <segment>
-<pinref part="C10" gate="G$1" pin="1"/>
+<pinref part="C10" gate="G$1" pin="+"/>
 <wire x1="-33.02" y1="152.4" x2="-30.48" y2="152.4" width="0.1524" layer="91"/>
 <label x="-25.4" y="154.94" size="1.778" layer="95"/>
@@
 <pinref part="U9" gate="G$1" pin="IN"/>
 <wire x1="-7.62" y1="137.16" x2="2.54" y2="137.16" width="0.1524" layer="91"/>
+<pinref part="C11" gate="G$1" pin="1"/>
 </segment>
 <segment>
@@
 <pinref part="JP2" gate="A" pin="3"/>
 <wire x1="167.64" y1="106.68" x2="177.8" y2="106.68" width="0.1524" layer="91"/>
-<pinref part="C16" gate="G$1" pin="1"/>
+<pinref part="C16" gate="G$1" pin="+"/>
 <wire x1="162.56" y1="96.52" x2="162.56" y2="91.44" width="0.1524" layer="91"/>
 <junction x="162.56" y="96.52"/>

Commit message: Added mount holes
Connections:
- net GND: now also JP2.3
- net N$16: now also JP2.4; no longer JP2.3
Changed lines of the file:
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@@
 <part name="R5" library="rcl-dhs" deviceset="R-US_" device="R0603" value="750"/>
 <part name="C11" library="rcl-dhs" deviceset="C-US" device="C0603" value=".1u"/>
+<part name="SUPPLY9" library="supply2" deviceset="GND" device=""/>
 </parts>
 <sheets>
@@
 <instance part="R5" gate="G$1" x="-127" y="68.58" rot="R180"/>
 <instance part="C11" gate="G$1" x="-33.02" y="149.86"/>
+<instance part="SUPPLY9" gate="GND" x="172.72" y="91.44"/>
 </instances>
 <busses>
@@
 <pinref part="SUPPLY8" gate="GND" pin="GND"/>
 <wire x1="162.56" y1="83.82" x2="162.56" y2="81.28" width="0.1524" layer="91"/>
+</segment>
+<segment>
+<pinref part="JP2" gate="A" pin="3"/>
+<wire x1="177.8" y1="106.68" x2="170.18" y2="106.68" width="0.1524" layer="91"/>
+<wire x1="170.18" y1="106.68" x2="170.18" y2="99.06" width="0.1524" layer="91"/>
+<pinref part="SUPPLY9" gate="GND" pin="GND"/>
+<wire x1="170.18" y1="99.06" x2="172.72" y2="99.06" width="0.1524" layer="91"/>
+<wire x1="172.72" y1="99.06" x2="172.72" y2="93.98" width="0.1524" layer="91"/>
 </segment>
 </net>
@@
 <wire x1="152.4" y1="96.52" x2="162.56" y2="96.52" width="0.1524" layer="91"/>
 <wire x1="162.56" y1="96.52" x2="167.64" y2="96.52" width="0.1524" layer="91"/>
-<wire x1="167.64" y1="96.52" x2="167.64" y2="106.68" width="0.1524" layer="91"/>
-<pinref part="JP2" gate="A" pin="3"/>
-<wire x1="167.64" y1="106.68" x2="177.8" y2="106.68" width="0.1524" layer="91"/>
 <pinref part="C16" gate="G$1" pin="+"/>
 <wire x1="162.56" y1="96.52" x2="162.56" y2="91.44" width="0.1524" layer="91"/>
 <junction x="162.56" y="96.52"/>
-</segment>
-</net>
+<pinref part="JP2" gate="A" pin="4"/>
+<wire x1="177.8" y1="104.14" x2="167.64" y2="104.14" width="0.1524" layer="91"/>
+<wire x1="167.64" y1="104.14" x2="167.64" y2="96.52" width="0.1524" layer="91"/>
+</segment>
+</net>

Commit message: layout tweaks
Connections:
- net N$12: no longer SJ10.1
- net N$16: now also SJ10.1
Other:
- moved on the sheet: SJ11
Changed lines of the file:
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@@
 <instance part="SJ9" gate="1" x="147.32" y="114.3"/>
 <instance part="SJ10" gate="1" x="147.32" y="106.68"/>
-<instance part="SJ11" gate="1" x="147.32" y="99.06"/>
+<instance part="SJ11" gate="1" x="142.24" y="86.36"/>
 <instance part="+3V7" gate="G$1" x="165.1" y="114.3" rot="R270"/>
 <instance part="P+3" gate="1" x="162.56" y="101.6" rot="R270"/>
@@
 <wire x1="119.38" y1="116.84" x2="142.24" y2="116.84" width="0.1524" layer="91"/>
 <wire x1="142.24" y1="116.84" x2="142.24" y2="114.3" width="0.1524" layer="91"/>
-<pinref part="SJ10" gate="1" pin="1"/>
-<wire x1="142.24" y1="106.68" x2="142.24" y2="114.3" width="0.1524" layer="91"/>
-<junction x="142.24" y="114.3"/>
-<pinref part="SJ11" gate="1" pin="1"/>
-<wire x1="142.24" y1="99.06" x2="142.24" y2="106.68" width="0.1524" layer="91"/>
-<junction x="142.24" y="106.68"/>
 <pinref part="C12" gate="G$1" pin="2"/>
 <wire x1="111.76" y1="137.16" x2="119.38" y2="137.16" width="0.1524" layer="91"/>
@@
 <wire x1="137.16" y1="137.16" x2="152.4" y2="137.16" width="0.1524" layer="91"/>
 <junction x="137.16" y="137.16"/>
+<wire x1="142.24" y1="114.3" x2="137.16" y2="114.3" width="0.1524" layer="91"/>
+<wire x1="137.16" y1="114.3" x2="137.16" y2="86.36" width="0.1524" layer="91"/>
+<junction x="142.24" y="114.3"/>
+<pinref part="SJ11" gate="1" pin="1"/>
 </segment>
 </net>
@@
 <segment>
 <pinref part="SJ11" gate="1" pin="2"/>
-<wire x1="152.4" y1="96.52" x2="152.4" y2="99.06" width="0.1524" layer="91"/>
+<wire x1="152.4" y1="96.52" x2="147.32" y2="86.36" width="0.1524" layer="91"/>
 <wire x1="152.4" y1="96.52" x2="162.56" y2="96.52" width="0.1524" layer="91"/>
 <wire x1="162.56" y1="96.52" x2="167.64" y2="96.52" width="0.1524" layer="91"/>
@@
 <wire x1="177.8" y1="104.14" x2="167.64" y2="104.14" width="0.1524" layer="91"/>
 <wire x1="167.64" y1="104.14" x2="167.64" y2="96.52" width="0.1524" layer="91"/>
-</segment>
-</net>
+<pinref part="SJ10" gate="1" pin="1"/>
+<wire x1="142.24" y1="106.68" x2="142.24" y2="96.52" width="0.1524" layer="91"/>
+<wire x1="142.24" y1="96.52" x2="152.4" y2="96.52" width="0.1524" layer="91"/>
+<junction x="152.4" y="96.52"/>
+</segment>
+</net>

Commit message: Tidy up and update pdf
Connections:
- net N$12 renamed VCCIO
Other:
- moved on the sheet: C10, C11, C12, C13, C14, C15, R1, R3, R5, SJ10, SJ11, SJ6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

Commit message: Board tweaks and added gerbers
Parts:
- SJ10, SJ11, SJ12, SJ9: value (none) -> JUMPER; device jumper:SJ -> rcl-dhs:JUMPER
